File: WIP/KiCad/cicadav1.kicad_pcb (KiCad board)
At the start: 2 copper layers, 281.5 x 153.9 mm, 67 parts

Commit message: config.yaml updated & testpcb from ergogen
Parts:
- moved MCU1 28.8 mm to (129.4, -51.7), turned to -90 degrees
Changed lines of the file:
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@@
   (page A3)
   (title_block
-    (title middle)
+    (title cicadav1)
     (rev 1)
     (company HagelzZ)
@@
         )
       (module ProMicro (layer F.Cu)
-      (at 153.5633113 -35.8790949 0)
+      (at 129.445495 -51.70757999999999 -90)
       (fp_text reference "MCU1" (at 0 0) (layer F.SilkS) hide (effects (font (size 1.27 1.27) (thickness 0.15))))
       (fp_text value "" (at 0 0) (layer F.SilkS) hide (effects (font (size 1.27 1.27) (thickness 0.15))))
@@
         (fp_line (start -15.24 6.35) (end -15.24 8.89) (layer F.SilkS) (width 0.15))
         (fp_line (start -12.7 6.35) (end -12.7 8.89) (layer F.SilkS) (width 0.15))
-        (fp_text user RAW (at -13.97 4.8 90) (layer F.SilkS) (effects (font (size 0.8 0.8) (thickness 0.15))))
-        (fp_text user GND (at -11.43 4.8 90) (layer F.SilkS) (effects (font (size 0.8 0.8) (thickness 0.15))))
-        (fp_text user RST (at -8.89 4.8 90) (layer F.SilkS) (effects (font (size 0.8 0.8) (thickness 0.15))))
-        (fp_text user VCC (at -6.35 4.8 90) (layer F.SilkS) (effects (font (size 0.8 0.8) (thickness 0.15))))
-        (fp_text user P21 (at -3.81 4.8 90) (layer F.SilkS) (effects (font (size 0.8 0.8) (thickness 0.15))))
-        (fp_text user P20 (at -1.27 4.8 90) (layer F.SilkS) (effects (font (size 0.8 0.8) (thickness 0.15))))
-        (fp_text user P19 (at 1.27 4.8 90) (layer F.SilkS) (effects (font (size 0.8 0.8) (thickness 0.15))))
-        (fp_text user P18 (at 3.81 4.8 90) (layer F.SilkS) (effects (font (size 0.8 0.8) (thickness 0.15))))
-        (fp_text user P15 (at 6.35 4.8 90) (layer F.SilkS) (effects (font (size 0.8 0.8) (thickness 0.15))))
-        (fp_text user P14 (at 8.89 4.8 90) (layer F.SilkS) (effects (font (size 0.8 0.8) (thickness 0.15))))
-        (fp_text user P16 (at 11.43 4.8 90) (layer F.SilkS) (effects (font (size 0.8 0.8) (thickness 0.15))))
-        (fp_text user P10 (at 13.97 4.8 90) (layer F.SilkS) (effects (font (size 0.8 0.8) (thickness 0.15))))
-        (fp_text user P01 (at -13.97 -4.8 90) (layer F.SilkS) (effects (font (size 0.8 0.8) (thickness 0.15))))
-        (fp_text user P00 (at -11.43 -4.8 90) (layer F.SilkS) (effects (font (size 0.8 0.8) (thickness 0.15))))
-        (fp_text user GND (at -8.89 -4.8 90) (layer F.SilkS) (effects (font (size 0.8 0.8) (thickness 0.15))))
-        (fp_text user GND (at -6.35 -4.8 90) (layer F.SilkS) (effects (font (size 0.8 0.8) (thickness 0.15))))
-        (fp_text user P02 (at -3.81 -4.8 90) (layer F.SilkS) (effects (font (size 0.8 0.8) (thickness 0.15))))
-        (fp_text user P03 (at -1.27 -4.8 90) (layer F.SilkS) (effects (font (size 0.8 0.8) (thickness 0.15))))
-        (fp_text user P04 (at 1.27 -4.8 90) (layer F.SilkS) (effects (font (size 0.8 0.8) (thickness 0.15))))
-        (fp_text user P05 (at 3.81 -4.8 90) (layer F.SilkS) (effects (font (size 0.8 0.8) (thickness 0.15))))
-        (fp_text user P06 (at 6.35 -4.8 90) (layer F.SilkS) (effects (font (size 0.8 0.8) (thickness 0.15))))
-        (fp_text user P07 (at 8.89 -4.8 90) (layer F.SilkS) (effects (font (size 0.8 0.8) (thickness 0.15))))
-        (fp_text user P08 (at 11.43 -4.8 90) (layer F.SilkS) (effects (font (size 0.8 0.8) (thickness 0.15))))
-        (fp_text user P09 (at 13.97 -4.8 90) (layer F.SilkS) (effects (font (size 0.8 0.8) (thickness 0.15))))
-        (pad 1 thru_hole rect (at -13.97 7.62 0) (size 1.7526 1.7526) (drill 1.0922) (layers *.Cu *.SilkS *.Mask) (net 67 "RAW"))
+        (fp_text user RAW (at -13.97 4.8 0) (layer F.SilkS) (effects (font (size 0.8 0.8) (thickness 0.15))))
+        (fp_text user GND (at -11.43 4.8 0) (layer F.SilkS) (effects (font (size 0.8 0.8) (thickness 0.15))))
+        (fp_text user RST (at -8.89 4.8 0) (layer F.SilkS) (effects (font (size 0.8 0.8) (thickness 0.15))))
+        (fp_text user VCC (at -6.35 4.8 0) (layer F.SilkS) (effects (font (size 0.8 0.8) (thickness 0.15))))
+        (fp_text user P21 (at -3.81 4.8 0) (layer F.SilkS) (effects (font (size 0.8 0.8) (thickness 0.15))))
+        (fp_text user P20 (at -1.27 4.8 0) (layer F.SilkS) (effects (font (size 0.8 0.8) (thickness 0.15))))
+        (fp_text user P19 (at 1.27 4.8 0) (layer F.SilkS) (effects (font (size 0.8 0.8) (thickness 0.15))))
+        (fp_text user P18 (at 3.81 4.8 0) (layer F.SilkS) (effects (font (size 0.8 0.8) (thickness 0.15))))
+        (fp_text user P15 (at 6.35 4.8 0) (layer F.SilkS) (effects (font (size 0.8 0.8) (thickness 0.15))))
+        (fp_text user P14 (at 8.89 4.8 0) (layer F.SilkS) (effects (font (size 0.8 0.8) (thickness 0.15))))
+        (fp_text user P16 (at 11.43 4.8 0) (layer F.SilkS) (effects (font (size 0.8 0.8) (thickness 0.15))))
+        (fp_text user P10 (at 13.97 4.8 0) (layer F.SilkS) (effects (font (size 0.8 0.8) (thickness 0.15))))
+        (fp_text user P01 (at -13.97 -4.8 0) (layer F.SilkS) (effects (font (size 0.8 0.8) (thickness 0.15))))
+        (fp_text user P00 (at -11.43 -4.8 0) (layer F.SilkS) (effects (font (size 0.8 0.8) (thickness 0.15))))
+        (fp_text user GND (at -8.89 -4.8 0) (layer F.SilkS) (effects (font (size 0.8 0.8) (thickness 0.15))))
+        (fp_text user GND (at -6.35 -4.8 0) (layer F.SilkS) (effects (font (size 0.8 0.8) (thickness 0.15))))
+        (fp_text user P02 (at -3.81 -4.8 0) (layer F.SilkS) (effects (font (size 0.8 0.8) (thickness 0.15))))
+        (fp_text user P03 (at -1.27 -4.8 0) (layer F.SilkS) (effects (font (size 0.8 0.8) (thickness 0.15))))
+        (fp_text user P04 (at 1.27 -4.8 0) (layer F.SilkS) (effects (font (size 0.8 0.8) (thickness 0.15))))
+        (fp_text user P05 (at 3.81 -4.8 0) (layer F.SilkS) (effects (font (size 0.8 0.8) (thickness 0.15))))
+        (fp_text user P06 (at 6.35 -4.8 0) (layer F.SilkS) (effects (font (size 0.8 0.8) (thickness 0.15))))
+        (fp_text user P07 (at 8.89 -4.8 0) (layer F.SilkS) (effects (font (size 0.8 0.8) (thickness 0.15))))
+        (fp_text user P08 (at 11.43 -4.8 0) (layer F.SilkS) (effects (font (size 0.8 0.8) (thickness 0.15))))
+        (fp_text user P09 (at 13.97 -4.8 0) (layer F.SilkS) (effects (font (size 0.8 0.8) (thickness 0.15))))
+        (pad 1 thru_hole rect (at -13.97 7.62 -90) (size 1.7526 1.7526) (drill 1.0922) (layers *.Cu *.SilkS *.Mask) (net 67 "RAW"))
         (pad 2 thru_hole circle (at -11.43 7.62 0) (size 1.7526 1.7526) (drill 1.0922) (layers *.Cu *.SilkS *.Mask) (net 68 "GND"))
         (pad 3 thru_hole circle (at -8.89 7.62 0) (size 1.7526 1.7526) (drill 1.0922) (layers *.Cu *.SilkS *.Mask) (net 69 "RST"))

Commit message: config.yaml & pcb update
Parts:
- added D1: , ComboDiode, F.Cu at (99.1, 104.9)
- added D10: , ComboDiode, F.Cu at (131.5, 30.9)
- added D11: , ComboDiode, F.Cu at (138.2, 102.2)
- added D12: , ComboDiode, F.Cu at (141.5, 83.5)
- added D13: , ComboDiode, F.Cu at (144.8, 64.7)
- added D14: , ComboDiode, F.Cu at (148.1, 46.0)
- added D15: , ComboDiode, F.Cu at (151.4, 27.3)
- added D16: , ComboDiode, F.Cu at (157.8, 100.5)
- added D17: , ComboDiode, F.Cu at (161.1, 81.8)
- added D18: , ComboDiode, F.Cu at (164.4, 63.1)
- added D19: , ComboDiode, F.Cu at (167.7, 44.4)
- added D2: , ComboDiode, F.Cu at (102.4, 86.2)
- added D20: , ComboDiode, F.Cu at (171.0, 25.7)
- added D21: , ComboDiode, F.Cu at (175.3, 110.7)
- added D22: , ComboDiode, F.Cu at (178.6, 92.0)
- added D23: , ComboDiode, F.Cu at (181.9, 73.3)
- added D24: , ComboDiode, F.Cu at (185.2, 54.6)
- added D25: , ComboDiode, F.Cu at (188.5, 35.9)
- added D26: , ComboDiode, F.Cu at (193.6, 116.5)
- added D27: , ComboDiode, F.Cu at (196.9, 97.8)
- added D28: , ComboDiode, F.Cu at (200.2, 79.1)
- added D29: , ComboDiode, F.Cu at (203.5, 60.4)
- added D3: , ComboDiode, F.Cu at (105.7, 67.5)
- added D30: , ComboDiode, F.Cu at (206.8, 41.7)
- added D31: , ComboDiode, F.Cu at (169.1, 135.2)
- added D32: , ComboDiode, F.Cu at (185.4, 145.0)
- added D33: , ComboDiode, F.Cu at (201.7, 154.8)
- added D34: , ComboDiode, F.Cu at (359.8, 104.9)
- added D35: , ComboDiode, F.Cu at (356.5, 86.2)
- added D36: , ComboDiode, F.Cu at (353.2, 67.5)
- added D37: , ComboDiode, F.Cu at (349.9, 48.8)
- added D38: , ComboDiode, F.Cu at (346.6, 30.1)
- added D39: , ComboDiode, F.Cu at (340.6, 105.8)
- added D4: , ComboDiode, F.Cu at (109.0, 48.8)
- added D40: , ComboDiode, F.Cu at (337.3, 87.0)
- added D41: , ComboDiode, F.Cu at (334.0, 68.3)
- added D42: , ComboDiode, F.Cu at (330.7, 49.6)
- added D43: , ComboDiode, F.Cu at (327.4, 30.9)
- added D44: , ComboDiode, F.Cu at (320.7, 102.2)
- added D45: , ComboDiode, F.Cu at (317.4, 83.5)
- added D46: , ComboDiode, F.Cu at (314.1, 64.7)
- added D47: , ComboDiode, F.Cu at (310.8, 46.0)
- added D48: , ComboDiode, F.Cu at (307.5, 27.3)
- added D49: , ComboDiode, F.Cu at (301.1, 100.5)
- added D5: , ComboDiode, F.Cu at (112.3, 30.1)
- added D50: , ComboDiode, F.Cu at (297.8, 81.8)
- added D51: , ComboDiode, F.Cu at (294.5, 63.1)
- added D52: , ComboDiode, F.Cu at (291.2, 44.4)
- added D53: , ComboDiode, F.Cu at (287.9, 25.7)
- added D54: , ComboDiode, F.Cu at (283.6, 110.7)
- added D55: , ComboDiode, F.Cu at (280.3, 92.0)
- added D56: , ComboDiode, F.Cu at (277.0, 73.3)
- added D57: , ComboDiode, F.Cu at (273.7, 54.6)
- added D58: , ComboDiode, F.Cu at (270.4, 35.9)
- added D59: , ComboDiode, F.Cu at (265.3, 116.5)
- added D6: , ComboDiode, F.Cu at (118.3, 105.8)
- added D60: , ComboDiode, F.Cu at (262.0, 97.8)
- added D61: , ComboDiode, F.Cu at (258.7, 79.1)
- added D62: , ComboDiode, F.Cu at (255.4, 60.4)
- added D63: , ComboDiode, F.Cu at (252.1, 41.7)
- added D64: , ComboDiode, F.Cu at (289.7, 135.2)
- added D65: , ComboDiode, F.Cu at (273.5, 145.0)
- added D66: , ComboDiode, F.Cu at (257.2, 154.8)
- added D7: , ComboDiode, F.Cu at (121.6, 87.0)
- added D8: , ComboDiode, F.Cu at (124.9, 68.3)
- added D9: , ComboDiode, F.Cu at (128.2, 49.6)
- moved S16 141.4 mm to (158.7, 95.6)
- moved S49 141.4 mm to (300.2, 95.6)
- moved S24 141.4 mm to (186.0, 49.7)
- moved S32 141.4 mm to (188.0, 140.7)
- moved S35 141.4 mm to (355.6, 81.3)
- moved S61 141.4 mm to (257.9, 74.1)
- moved S53 141.4 mm to (287.0, 20.8)
- moved S56 141.4 mm to (276.1, 68.4)
- moved S43 141.4 mm to (326.6, 26.0)
- moved S46 141.4 mm to (313.2, 59.8)
- moved S5 141.4 mm to (113.2, 25.2)
- moved S12 141.4 mm to (142.4, 78.5)
- moved S19 141.4 mm to (168.5, 39.5)
- moved S33 141.4 mm to (204.3, 150.5)
- moved S40 141.4 mm to (336.4, 82.1)
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Connections:
- S21 pad 1: (no net) -> P20
- S22 pad 1: (no net) -> P20
- S23 pad 1: (no net) -> P20
- S24 pad 1: (no net) -> P20
- S25 pad 1: (no net) -> P20
- S26 pad 1: (no net) -> P21
- S27 pad 1: (no net) -> P21
- S28 pad 1: (no net) -> P21
- S29 pad 1: (no net) -> P21
- S30 pad 1: (no net) -> P21
- S54 pad 1: (no net) -> P0
- S55 pad 1: (no net) -> P0
- S56 pad 1: (no net) -> P0
- S57 pad 1: (no net) -> P0
- S58 pad 1: (no net) -> P0
- S59 pad 1: (no net) -> P1
- S60 pad 1: (no net) -> P1
- S61 pad 1: (no net) -> P1
- S62 pad 1: (no net) -> P1
- S63 pad 1: (no net) -> P1
Other:
- net class Default removed

Commit message: pcb and config.yaml update
Parts:
- moved MCU1 44.0 mm to (224.4, 90.4)
- moved D65 33.2 mm to (255.1, 172.7), turned to -59 degrees
- moved D66 33.2 mm to (238.9, 182.4), turned to -59 degrees
- moved D64 33.2 mm to (271.4, 162.9), turned to -59 degrees
- moved D61 30.8 mm to (240.0, 103.6), turned to -80 degrees
- moved D46 30.8 mm to (295.4, 89.3), turned to -80 degrees
- moved D53 30.8 mm to (269.2, 50.2), turned to -80 degrees
- moved D59 30.8 mm to (246.6, 141.0), turned to -80 degrees
- moved D58 30.8 mm to (251.7, 60.4), turned to -80 degrees
- moved D57 30.8 mm to (255.0, 79.1), turned to -80 degrees
- moved D51 30.8 mm to (275.8, 87.6), turned to -80 degrees
- moved D44 30.8 mm to (302.0, 126.7), turned to -80 degrees
- moved D50 30.8 mm to (279.1, 106.3), turned to -80 degrees
- moved D37 30.8 mm to (331.1, 73.3), turned to -80 degrees
- moved D36 30.8 mm to (334.4, 92.0), turned to -80 degrees
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Other:
- board size 281.5 x 153.9 mm -> 273.8 x 156 mm
- net class Default added: clearance 0.2, trace_width 0.25, via_dia 0.8, via_drill 0.4

Commit message: config and pcb update
Parts:
- moved D39 30.4 mm to (331.2, 159.2), turned to 10 degrees
- moved D6 30.4 mm to (117.7, 159.2), turned to -10 degrees
- moved D7 30.4 mm to (121.0, 140.5), turned to -10 degrees
- moved D11 30.4 mm to (137.6, 155.6), turned to -10 degrees
- moved D12 30.4 mm to (140.9, 136.9), turned to -10 degrees
- moved D40 30.4 mm to (327.9, 140.5), turned to 10 degrees
- moved D44 30.4 mm to (311.3, 155.6), turned to 10 degrees
- moved D45 30.4 mm to (308.0, 136.9), turned to 10 degrees
- moved D10 30.4 mm to (130.9, 84.4), turned to -10 degrees
- moved D15 30.4 mm to (150.8, 80.8), turned to -10 degrees
- moved D43 30.4 mm to (318.0, 84.4), turned to 10 degrees
- moved D48 30.4 mm to (298.1, 80.8), turned to 10 degrees
- moved D1 30.4 mm to (98.5, 158.4), turned to -10 degrees
- moved D13 30.4 mm to (144.2, 118.2), turned to -10 degrees
- moved D14 30.4 mm to (147.5, 99.5), turned to -10 degrees
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Other:
- board size 273.8 x 156 mm -> 275.6 x 158 mm

Commit message: keyb update
Parts:
- moved D10 4.00 mm to (130.2, 88.3)
- moved D15 4.00 mm to (150.1, 84.7)
- moved D20 4.00 mm to (169.7, 83.1)
- moved D25 4.00 mm to (187.2, 93.3)
- moved D30 4.00 mm to (205.5, 99.0)
- moved D5 4.00 mm to (111.0, 87.5)
- moved S10 4.00 mm to (131.6, 79.9)
- moved S15 4.00 mm to (151.6, 76.3)
- moved S20 4.00 mm to (171.2, 74.7)
- moved S25 4.00 mm to (188.7, 84.9)
- moved S30 4.00 mm to (206.9, 90.7)
- moved S5 4.00 mm to (112.5, 79.1)
- moved D38 3.95 mm to (337.5, 87.5)
- moved D43 3.95 mm to (318.4, 88.3)
- moved D48 3.95 mm to (298.4, 84.7)
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Connections:
- S21 pad 1: P20 -> (no net)
- S22 pad 1: P20 -> (no net)
- S23 pad 1: P20 -> (no net)
- S24 pad 1: P20 -> (no net)
- S25 pad 1: P20 -> (no net)
- S26 pad 1: P21 -> (no net)
- S27 pad 1: P21 -> (no net)
- S28 pad 1: P21 -> (no net)
- S29 pad 1: P21 -> (no net)
- S30 pad 1: P21 -> (no net)
- S31 pad 1: (no net) -> P19
- S32 pad 1: (no net) -> P20
- S33 pad 1: (no net) -> P21
- S54 pad 1: P0 -> (no net)
- S55 pad 1: P0 -> (no net)
- S56 pad 1: P0 -> (no net)
- S57 pad 1: P0 -> (no net)
- S58 pad 1: P0 -> (no net)
- S59 pad 1: P1 -> (no net)
- S60 pad 1: P1 -> (no net)
- S61 pad 1: P1 -> (no net)
- S62 pad 1: P1 -> (no net)
- S63 pad 1: P1 -> (no net)
- S64 pad 1: (no net) -> P19
- S65 pad 1: (no net) -> P20
- S66 pad 1: (no net) -> P21
Other:
- board size 275.6 x 158 mm -> 275.2 x 154.1 mm

Commit message: yupdate
Connections:
- D1 pad 1: (no net) -> P15
- D10 pad 1: (no net) -> P21
- D11 pad 1: (no net) -> P15
- D12 pad 1: (no net) -> P18
- D13 pad 1: (no net) -> P19
- D14 pad 1: (no net) -> P20
- D15 pad 1: (no net) -> P21
- D16 pad 1: (no net) -> P15
- D17 pad 1: (no net) -> P18
- D18 pad 1: (no net) -> P19
- D19 pad 1: (no net) -> P20
- D2 pad 1: (no net) -> P18
- D20 pad 1: (no net) -> P21
- D21 pad 1: (no net) -> P15
- D22 pad 1: (no net) -> P18
- D23 pad 1: (no net) -> P19
- D24 pad 1: (no net) -> P20
- D25 pad 1: (no net) -> P21
- D26 pad 1: (no net) -> P15
- D27 pad 1: (no net) -> P18
- D28 pad 1: (no net) -> P19
- D29 pad 1: (no net) -> P20
- D3 pad 1: (no net) -> P19
- D30 pad 1: (no net) -> P21
- D31 pad 1: (no net) -> P9
- D32 pad 1: (no net) -> P9
- D33 pad 1: (no net) -> P9
- D34 pad 1: (no net) -> P15
- D35 pad 1: (no net) -> P18
- D36 pad 1: (no net) -> P19
- D37 pad 1: (no net) -> P20
- D38 pad 1: (no net) -> P21
- D39 pad 1: (no net) -> P15
- D4 pad 1: (no net) -> P20
- D40 pad 1: (no net) -> P18
- D41 pad 1: (no net) -> P19
- D42 pad 1: (no net) -> P20
- D43 pad 1: (no net) -> P21
- D44 pad 1: (no net) -> P15
- D45 pad 1: (no net) -> P18
- D46 pad 1: (no net) -> P19
- D47 pad 1: (no net) -> P20
- D48 pad 1: (no net) -> P21
- D49 pad 1: (no net) -> P15
- D5 pad 1: (no net) -> P21
- D50 pad 1: (no net) -> P18
- D51 pad 1: (no net) -> P19
- D52 pad 1: (no net) -> P20
- D53 pad 1: (no net) -> P21
- D54 pad 1: (no net) -> P15
- D55 pad 1: (no net) -> P18
- D56 pad 1: (no net) -> P19
- D57 pad 1: (no net) -> P20
- D58 pad 1: (no net) -> P21
- D59 pad 1: (no net) -> P15
- D6 pad 1: (no net) -> P15
- D60 pad 1: (no net) -> P18
- D61 pad 1: (no net) -> P19
- D62 pad 1: (no net) -> P20
- D63 pad 1: (no net) -> P21
- D64 pad 1: (no net) -> P8
- D65 pad 1: (no net) -> P8
- D66 pad 1: (no net) -> P8
- D7 pad 1: (no net) -> P18
- D8 pad 1: (no net) -> P19
- D9 pad 1: (no net) -> P20

Commit message: oopdade
Parts:
- moved D1 0.50 mm to (98.4, 158.9)
- moved D10 0.50 mm to (130.1, 88.8)
- moved D11 0.50 mm to (137.5, 156.1)
- moved D12 0.50 mm to (140.6, 138.4)
- moved D13 0.50 mm to (143.8, 120.7)
- moved D14 0.50 mm to (146.9, 102.9)
- moved D15 0.50 mm to (150.0, 85.2)
- moved D16 0.50 mm to (157.1, 154.5)
- moved D17 0.50 mm to (160.2, 136.8)
- moved D18 0.50 mm to (163.3, 119.0)
- moved D19 0.50 mm to (166.5, 101.3)
- moved D2 0.50 mm to (101.6, 141.1)
- moved D20 0.50 mm to (169.6, 83.6)
- moved D21 0.50 mm to (174.6, 164.7)
- moved D22 0.50 mm to (177.7, 146.9)
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Connections:
- D1 pad 1: P15 -> P16
- D10 pad 1: P21 -> P19
- D11 pad 1: P15 -> P16
- D12 pad 1: P18 -> P14
- D13 pad 1: P19 -> P15
- D14 pad 1: P20 -> P18
- D15 pad 1: P21 -> P19
- D16 pad 1: P15 -> P16
- D17 pad 1: P18 -> P14
- D18 pad 1: P19 -> P15
- D19 pad 1: P20 -> P18
- D2 pad 1: P18 -> P14
- D20 pad 1: P21 -> P19
- D21 pad 1: P15 -> P16
- D22 pad 1: P18 -> P14
- D23 pad 1: P19 -> P15
- D24 pad 1: P20 -> P18
- D25 pad 1: P21 -> P19
- D26 pad 1: P15 -> P16
- D27 pad 1: P18 -> P14
- D28 pad 1: P19 -> P15
- D29 pad 1: P20 -> P18
- D3 pad 1: P19 -> P15
- D30 pad 1: P21 -> P19
- D31 pad 1: P9 -> P10
- D32 pad 1: P9 -> P10
- D33 pad 1: P9 -> P10
- D34 pad 1: P15 -> P8
- D35 pad 1: P18 -> P7
- D36 pad 1: P19 -> P6
- D37 pad 1: P20 -> P5
- D38 pad 1: P21 -> P4
- D39 pad 1: P15 -> P8
- D4 pad 1: P20 -> P18
- D40 pad 1: P18 -> P7
- D41 pad 1: P19 -> P6
- D42 pad 1: P20 -> P5
- D43 pad 1: P21 -> P4
- D44 pad 1: P15 -> P8
- D45 pad 1: P18 -> P7
- D46 pad 1: P19 -> P6
- D47 pad 1: P20 -> P5
- D48 pad 1: P21 -> P4
- D49 pad 1: P15 -> P8
- D5 pad 1: P21 -> P19
- D50 pad 1: P18 -> P7
- D51 pad 1: P19 -> P6
- D52 pad 1: P20 -> P5
- D53 pad 1: P21 -> P4
- D54 pad 1: P15 -> P8
- D55 pad 1: P18 -> P7
- D56 pad 1: P19 -> P6
- D57 pad 1: P20 -> P5
- D58 pad 1: P21 -> P4
- D59 pad 1: P15 -> P8
- D6 pad 1: P15 -> P16
- D60 pad 1: P18 -> P7
- D61 pad 1: P19 -> P6
- D62 pad 1: P20 -> P5
- D63 pad 1: P21 -> P4
- D64 pad 1: P8 -> P9
- D65 pad 1: P8 -> P9
- D66 pad 1: P8 -> P9
- D7 pad 1: P18 -> P14
- D8 pad 1: P19 -> P15
- D9 pad 1: P20 -> P18
- S31 pad 1: P19 -> (no net)
- S32 pad 1: P20 -> (no net)
- S33 pad 1: P21 -> (no net)
- S64 pad 1: P19 -> (no net)
- S65 pad 1: P20 -> (no net)
- S66 pad 1: P21 -> (no net)

Commit message: config + pcb update
Connections:
- S1 pad 1: (no net) -> P20
- S10 pad 1: (no net) -> P21
- S11 pad 1: (no net) -> P3
- S12 pad 1: (no net) -> P3
- S13 pad 1: (no net) -> P3
- S14 pad 1: (no net) -> P3
- S15 pad 1: (no net) -> P3
- S16 pad 1: (no net) -> P2
- S17 pad 1: (no net) -> P2
- S18 pad 1: (no net) -> P2
- S19 pad 1: (no net) -> P2
- S2 pad 1: (no net) -> P20
- S20 pad 1: (no net) -> P2
- S21 pad 1: (no net) -> P0
- S22 pad 1: (no net) -> P0
- S23 pad 1: (no net) -> P0
- S24 pad 1: (no net) -> P0
- S25 pad 1: (no net) -> P0
- S26 pad 1: (no net) -> P1
- S27 pad 1: (no net) -> P1
- S28 pad 1: (no net) -> P1
- S29 pad 1: (no net) -> P1
- S3 pad 1: (no net) -> P20
- S30 pad 1: (no net) -> P1
- S31 pad 1: (no net) -> P2
- S32 pad 1: (no net) -> P0
- S33 pad 1: (no net) -> P1
- S34 pad 1: (no net) -> P20
- S35 pad 1: (no net) -> P20
- S36 pad 1: (no net) -> P20
- S37 pad 1: (no net) -> P20
- S38 pad 1: (no net) -> P20
- S39 pad 1: (no net) -> P21
- S4 pad 1: (no net) -> P20
- S40 pad 1: (no net) -> P21
- S41 pad 1: (no net) -> P21
- S42 pad 1: (no net) -> P21
- S43 pad 1: (no net) -> P21
- S44 pad 1: (no net) -> P3
- S45 pad 1: (no net) -> P3
- S46 pad 1: (no net) -> P3
- S47 pad 1: (no net) -> P3
- S48 pad 1: (no net) -> P3
- S49 pad 1: (no net) -> P2
- S5 pad 1: (no net) -> P20
- S50 pad 1: (no net) -> P2
- S51 pad 1: (no net) -> P2
- S52 pad 1: (no net) -> P2
- S53 pad 1: (no net) -> P2
- S54 pad 1: (no net) -> P0
- S55 pad 1: (no net) -> P0
- S56 pad 1: (no net) -> P0
- S57 pad 1: (no net) -> P0
- S58 pad 1: (no net) -> P0
- S59 pad 1: (no net) -> P1
- S6 pad 1: (no net) -> P21
- S60 pad 1: (no net) -> P1
- S61 pad 1: (no net) -> P1
- S62 pad 1: (no net) -> P1
- S63 pad 1: (no net) -> P1
- S64 pad 1: (no net) -> P2
- S65 pad 1: (no net) -> P0
- S66 pad 1: (no net) -> P1
- S7 pad 1: (no net) -> P21
- S8 pad 1: (no net) -> P21
- S9 pad 1: (no net) -> P21
