File: WIP/KiCad/cicadav1.kicad_pcb (KiCad board)
At the start: 2 copper layers, 275.2 x 154.1 mm, 133 parts

Commit message: config + gitignore + pcb update
Parts:
- moved MCU1 3.50 mm to (224.3, 119.9)
Changed lines of the file:
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@@
     )
       (module ProMicro (layer F.Cu)
-      (at 224.2734178 123.39291930000002 -90)
+      (at 224.2734178 119.89291930000002 -90)
       (fp_text reference "MCU1" (at 0 0) (layer F.SilkS) hide (effects (font (size 1.27 1.27) (thickness 0.15))))
       (fp_text value "" (at 0 0) (layer F.SilkS) hide (effects (font (size 1.27 1.27) (thickness 0.15))))

Commit message: pcb update
Parts:
- moved D1 128.5 mm to (226.3, 171.8), turned to -100 degrees
- moved D2 128.5 mm to (229.3, 154.8), turned to -100 degrees
- moved D3 128.3 mm to (232.0, 139.7), turned to -100 degrees
- moved D6 107.2 mm to (224.1, 171.4), turned to -100 degrees
- moved D7 107.1 mm to (227.1, 154.4), turned to -100 degrees
- moved D8 107.0 mm to (229.8, 139.3), turned to -100 degrees
- moved D34 104.2 mm to (246.7, 171.6), turned to -80 degrees
- moved D35 104.1 mm to (243.8, 155.1), turned to -80 degrees
- moved D36 103.9 mm to (241.2, 139.7), turned to -80 degrees
- moved D13 85.7 mm to (227.5, 138.9), turned to -100 degrees
- moved D12 85.7 mm to (224.9, 154.0), turned to -100 degrees
- moved D11 85.7 mm to (221.9, 171.0), turned to -100 degrees
- moved D39 82.8 mm to (248.9, 171.2), turned to -80 degrees
- moved D40 82.8 mm to (246.0, 154.7), turned to -80 degrees
- moved D41 82.7 mm to (243.4, 139.3), turned to -80 degrees
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Routing:
- net P20: track 0.00 -> 510.1 mm, vias 0 -> 6
- net P21: track 0.00 -> 495.4 mm, vias 0 -> 6
- net P2: track 0.00 -> 494.5 mm, vias 0 -> 13
- net P3: track 0.00 -> 469.4 mm, vias 0 -> 9
- net P0: track 0.00 -> 447.6 mm, vias 0 -> 13
- net P1: track 0.00 -> 423.3 mm, vias 0 -> 15
- net mirror_outer_top: track 0.00 -> 159.3 mm, vias 0 -> 1
- net mirror_outer_home: track 0.00 -> 158.9 mm, vias 0 -> 1
- net mirror_outer_bottom: track 0.00 -> 153.7 mm, vias 0 -> 1
- net P19: track 0.00 -> 138.7 mm
- net mirror_pinky_top: track 0.00 -> 137.2 mm, vias 0 -> 1
- net mirror_pinky_home: track 0.00 -> 136.5 mm, vias 0 -> 1
- net P4: track 0.00 -> 133.4 mm
- net outer_home: track 0.00 -> 133.4 mm, vias 0 -> 7
- net mirror_pinky_bottom: track 0.00 -> 131.6 mm, vias 0 -> 1
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Other:
- net class Default removed
